File: Orentation2.kicad_sch (KiCad schematic)
At the start: 12 parts, among them U1 LotsOfPins, U10 LotsOfPins, U11 LotsOfPins, U12 LotsOfPins, U2 LotsOfPins, U3 LotsOfPins, U4 LotsOfPins, U5 LotsOfPins, U6 LotsOfPins, U7 LotsOfPins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

Commit message: symbol instance name/number hiding
Parts:
- added U? (x3): LotsOfPins, symbol Orientation2Lib:LotsOfPins
Other:
- note added: "Hide Both"
- note added: "Hide Names"
- note added: "Hide Numbers"
Changed lines of the file:
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@@
+    (effects (font (size 1.27 1.27)) (justify left bottom))
+  )
+  (text "Hide Numbers" (at 243.84 16.51 0)
     (effects (font (size 1.27 1.27)) (justify left bottom))
   )
@@
     (effects (font (size 1.27 1.27)) (justify left bottom))
   )
+  (text "Hide Names" (at 245.11 60.96 0)
+    (effects (font (size 1.27 1.27)) (justify left bottom))
+  )
   (text "+90" (at 38.1 76.2 0)
+    (effects (font (size 1.27 1.27)) (justify left bottom))
+  )
+  (text "Hide Both" (at 245.11 104.14 0)
     (effects (font (size 1.27 1.27)) (justify left bottom))
   )
@@
     (pin "1")
     (pin "10")
-    (pin "19")
-    (pin "28")
-    (pin "2")
-    (pin "11")
-    (pin "20")
-    (pin "29")
-    (pin "3")
-    (pin "12")
-    (pin "21")
-    (pin "30")
-    (pin "4")
-    (pin "13")
-    (pin "22")
-    (pin "31")
-    (pin "5")
-    (pin "14")
-    (pin "23")
-    (pin "32")
-    (pin "6")
-    (pin "33")
-    (pin "15")
-    (pin "24")
-    (pin "7")
-    (pin "34")
-    (pin "16")
-    (pin "25")
-    (pin "8")
-    (pin "35")
-    (pin "17")
-    (pin "26")
-    (pin "9")
-    (pin "36")
-    (pin "18")
-    (pin "27")
+    (pin "11")
+    (pin "12")
+    (pin "13")
+    (pin "14")
+    (pin "15")
+    (pin "16")
+    (pin "17")
+    (pin "18")
+    (pin "19")
+    (pin "2")
+    (pin "20")
+    (pin "21")
+    (pin "22")
+    (pin "23")
+    (pin "24")
+    (pin "25")
+    (pin "26")
+    (pin "27")
+    (pin "28")
+    (pin "29")
+    (pin "3")
+    (pin "30")
+    (pin "31")
+    (pin "32")
+    (pin "33")
+    (pin "34")
+    (pin "35")
+    (pin "36")
+    (pin "4")
+    (pin "5")
+    (pin "6")
+    (pin "7")
+    (pin "8")
+    (pin "9")
+  )
+  (symbol (lib_name "LotsOfPins_2") (lib_id "Orientation2Lib:LotsOfPins") (at 266.7 85.09 0) (unit 1)
+    (in_bom yes) (on_board yes) (fields_autoplaced)
+    (property "Reference" "U?" (id 0) (at 281.94 60.7312 0))
+    (property "Value" "LotsOfPins" (id 1) (at 281.94 63.2712 0))
+    (property "Footprint" "" (id 2) (at 266.7 85.09 0)
+      (effects (font (size 1.27 1.27)) hide)
+    )
+    (property "Datasheet" "" (id 3) (at 266.7 85.09 0)
+      (effects (font (size 1.27 1.27)) hide)
+    )
+    (pin "1")
+    (pin "10")
+    (pin "11")
+    (pin "12")
+    (pin "13")
+    (pin "14")
+    (pin "15")
+    (pin "16")
+    (pin "17")
+    (pin "18")
+    (pin "19")
+    (pin "2")
+    (pin "20")
+    (pin "21")
+    (pin "22")
+    (pin "23")
+    (pin "24")
+    (pin "25")
+    (pin "26")
+    (pin "27")
+    (pin "28")
+    (pin "29")
+    (pin "3")
+    (pin "30")
+    (pin "31")
+    (pin "32")
+    (pin "33")
+    (pin "34")
+    (pin "35")
+    (pin "36")
+    (pin "4")
+    (pin "5")
+    (pin "6")
+    (pin "7")
+    (pin "8")
+    (pin "9")
   )
   (symbol (lib_id "Orientation2Lib:LotsOfPins") (at 196.85 160.02 0) (mirror x) (unit 1)
@@
     (pin "9")
   )
+  (symbol (lib_name "LotsOfPins_3") (lib_id "Orientation2Lib:LotsOfPins") (at 267.97 128.27 0) (unit 1)
+    (in_bom yes) (on_board yes) (fields_autoplaced)
+    (property "Reference" "U?" (id 0) (at 283.21 103.9112 0))
+    (property "Value" "LotsOfPins" (id 1) (at 283.21 106.4512 0))
+    (property "Footprint" "" (id 2) (at 267.97 128.27 0)
+      (effects (font (size 1.27 1.27)) hide)
+    )
+    (property "Datasheet" "" (id 3) (at 267.97 128.27 0)
+      (effects (font (size 1.27 1.27)) hide)
+    )
+    (pin "1")
+    (pin "10")
+    (pin "11")
+    (pin "12")
+    (pin "13")
+    (pin "14")
+    (pin "15")
+    (pin "16")
+    (pin "17")
+    (pin "18")
+    (pin "19")
+    (pin "2")
+    (pin "20")
+    (pin "21")
+    (pin "22")
+    (pin "23")
+    (pin "24")
+    (pin "25")
+    (pin "26")
+    (pin "27")
+    (pin "28")
+    (pin "29")
+    (pin "3")
+    (pin "30")
+    (pin "31")
+    (pin "32")
+    (pin "33")
+    (pin "34")
+    (pin "35")
+    (pin "36")
+    (pin "4")
+    (pin "5")
+    (pin "6")
+    (pin "7")
+    (pin "8")
+    (pin "9")
+  )
   (symbol (lib_id "Orientation2Lib:LotsOfPins") (at 73.66 69.85 90) (unit 1)
     (in_bom yes) (on_board yes) (fields_autoplaced)
@@
     (pin "9")
   )
+  (symbol (lib_name "LotsOfPins_1") (lib_id "Orientation2Lib:LotsOfPins") (at 266.7 40.64 0) (unit 1)
+    (in_bom yes) (on_board yes) (fields_autoplaced)
+    (property "Reference" "U?" (id 0) (at 281.94 16.2812 0))
+    (property "Value" "LotsOfPins" (id 1) (at 281.94 18.8212 0))
+    (property "Footprint" "" (id 2) (at 266.7 40.64 0)
+      (effects (font (size 1.27 1.27)) hide)
+    )
+    (property "Datasheet" "" (id 3) (at 266.7 40.64 0)
+      (effects (font (size 1.27 1.27)) hide)
+    )
+    (pin "1")
+    (pin "10")
+    (pin "11")
+    (pin "12")
+    (pin "13")
+    (pin "14")
+    (pin "15")
+    (pin "16")
+    (pin "17")
+    (pin "18")
+    (pin "19")
+    (pin "2")
+    (pin "20")
+    (pin "21")
+    (pin "22")
+    (pin "23")
+    (pin "24")
+    (pin "25")
+    (pin "26")
+    (pin "27")
+    (pin "28")
+    (pin "29")
+    (pin "3")
+    (pin "30")
+    (pin "31")
+    (pin "32")
+    (pin "33")
+    (pin "34")
+    (pin "35")
+    (pin "36")
+    (pin "4")
+    (pin "5")
+    (pin "6")
+    (pin "7")
+    (pin "8")
+    (pin "9")
+  )
   (symbol (lib_id "Orientation2Lib:LotsOfPins") (at 196.85 124.46 90) (mirror x) (unit 1)
     (in_bom yes) (on_board yes) (fields_autoplaced)
@@
       (reference "U12") (unit 1) (value "LotsOfPins") (footprint "")
     )
-  )
+    (path "/337b2738-ac74-46e4-af99-edf86290f598"
+      (reference "U?") (unit 1) (value "LotsOfPins") (footprint "")
+    )
+    (path "/a5b0d54e-9873-4c04-8e3b-2303e065a341"
+      (reference "U?") (unit 1) (value "LotsOfPins") (footprint "")
+    )
+    (path "/b364135e-c5d3-4ae8-be89-ca9a24a910d3"
+      (reference "U?") (unit 1) (value "LotsOfPins") (footprint "")
+    )
+  )

Commit message: more visibility test
Parts:
- added U13, U14, U15, U18: PinVis, symbol Orientation2Lib:PinVis
- gave numbers to parts that had none: 3
Other:
- note added: "Show Both"
- note added: "Show Names"
- note added: "Show Pins"
Changed lines of the file:
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@@
+    (effects (font (size 1.27 1.27)) (justify left bottom))
+  )
+  (text "Show Pins" (at 238.76 146.05 0)
+    (effects (font (size 1.27 1.27)) (justify left bottom))
+  )
+  (text "Show Both" (at 250.19 163.83 0)
     (effects (font (size 1.27 1.27)) (justify left bottom))
   )
@@
   )
   (text "Hide Names" (at 245.11 60.96 0)
+    (effects (font (size 1.27 1.27)) (justify left bottom))
+  )
+  (text "Show Names" (at 260.35 146.05 0)
     (effects (font (size 1.27 1.27)) (justify left bottom))
   )
@@
     (pin "9")
   )
+  (symbol (lib_name "PinVis_2") (lib_id "Orientation2Lib:PinVis") (at 266.7 153.67 0) (unit 1)
+    (in_bom yes) (on_board yes) (fields_autoplaced)
+    (property "Reference" "U18" (id 0) (at 274.32 148.971 0))
+    (property "Value" "PinVis" (id 1) (at 274.32 151.511 0))
+    (property "Footprint" "" (id 2) (at 264.795 152.4 0)
+      (effects (font (size 1.27 1.27)) hide)
+    )
+    (property "Datasheet" "" (id 3) (at 264.795 152.4 0)
+      (effects (font (size 1.27 1.27)) hide)
+    )
+    (pin "1")
+    (pin "2")
+    (pin "3")
+    (pin "4")
+  )
   (symbol (lib_id "Orientation2Lib:LotsOfPins") (at 73.66 39.37 0) (unit 1)
     (in_bom yes) (on_board yes) (fields_autoplaced)
@@
   (symbol (lib_name "LotsOfPins_2") (lib_id "Orientation2Lib:LotsOfPins") (at 266.7 85.09 0) (unit 1)
     (in_bom yes) (on_board yes) (fields_autoplaced)
-    (property "Reference" "U?" (id 0) (at 281.94 60.7312 0))
+    (property "Reference" "U17" (id 0) (at 281.94 60.7312 0))
     (property "Value" "LotsOfPins" (id 1) (at 281.94 63.2712 0))
     (property "Footprint" "" (id 2) (at 266.7 85.09 0)
@@
     (pin "8")
     (pin "9")
+  )
+  (symbol (lib_name "PinVis_3") (lib_id "Orientation2Lib:PinVis") (at 256.54 171.45 0) (unit 1)
+    (in_bom yes) (on_board yes) (fields_autoplaced)
+    (property "Reference" "U15" (id 0) (at 264.16 166.751 0))
+    (property "Value" "PinVis" (id 1) (at 264.16 169.291 0))
+    (property "Footprint" "" (id 2) (at 254.635 170.18 0)
+      (effects (font (size 1.27 1.27)) hide)
+    )
+    (property "Datasheet" "" (id 3) (at 254.635 170.18 0)
+      (effects (font (size 1.27 1.27)) hide)
+    )
+    (pin "1")
+    (pin "2")
+    (pin "3")
+    (pin "4")
   )
   (symbol (lib_id "Orientation2Lib:LotsOfPins") (at 196.85 160.02 0) (mirror x) (unit 1)
@@
     (pin "9")
   )
+  (symbol (lib_id "Orientation2Lib:PinVis") (at 224.79 153.67 0) (unit 1)
+    (in_bom yes) (on_board yes) (fields_autoplaced)
+    (property "Reference" "U13" (id 0) (at 232.41 148.971 0))
+    (property "Value" "PinVis" (id 1) (at 232.41 151.511 0))
+    (property "Footprint" "" (id 2) (at 222.885 152.4 0)
+      (effects (font (size 1.27 1.27)) hide)
+    )
+    (property "Datasheet" "" (id 3) (at 222.885 152.4 0)
+      (effects (font (size 1.27 1.27)) hide)
+    )
+    (pin "1")
+    (pin "2")
+    (pin "3")
+    (pin "4")
+  )
   (symbol (lib_id "Orientation2Lib:LotsOfPins") (at 123.19 115.57 270) (mirror x) (unit 1)
     (in_bom yes) (on_board yes) (fields_autoplaced)
@@
   (symbol (lib_name "LotsOfPins_3") (lib_id "Orientation2Lib:LotsOfPins") (at 267.97 128.27 0) (unit 1)
     (in_bom yes) (on_board yes) (fields_autoplaced)
-    (property "Reference" "U?" (id 0) (at 283.21 103.9112 0))
+    (property "Reference" "U19" (id 0) (at 283.21 103.9112 0))
     (property "Value" "LotsOfPins" (id 1) (at 283.21 106.4512 0))
     (property "Footprint" "" (id 2) (at 267.97 128.27 0)
@@
   (symbol (lib_name "LotsOfPins_1") (lib_id "Orientation2Lib:LotsOfPins") (at 266.7 40.64 0) (unit 1)
     (in_bom yes) (on_board yes) (fields_autoplaced)
-    (property "Reference" "U?" (id 0) (at 281.94 16.2812 0))
+    (property "Reference" "U16" (id 0) (at 281.94 16.2812 0))
     (property "Value" "LotsOfPins" (id 1) (at 281.94 18.8212 0))
     (property "Footprint" "" (id 2) (at 266.7 40.64 0)
@@
     (pin "8")
     (pin "9")
+  )
+  (symbol (lib_name "PinVis_1") (lib_id "Orientation2Lib:PinVis") (at 246.38 153.67 0) (unit 1)
+    (in_bom yes) (on_board yes) (fields_autoplaced)
+    (property "Reference" "U14" (id 0) (at 254 148.971 0))
+    (property "Value" "PinVis" (id 1) (at 254 151.511 0))
+    (property "Footprint" "" (id 2) (at 244.475 152.4 0)
+      (effects (font (size 1.27 1.27)) hide)
+    )
+    (property "Datasheet" "" (id 3) (at 244.475 152.4 0)
+      (effects (font (size 1.27 1.27)) hide)
+    )
+    (pin "1")
+    (pin "2")
+    (pin "3")
+    (pin "4")
   )
   (symbol (lib_id "Orientation2Lib:LotsOfPins") (at 196.85 124.46 90) (mirror x) (unit 1)
@@
       (reference "U12") (unit 1) (value "LotsOfPins") (footprint "")
     )
+    (path "/630ab2b7-5d04-409d-8d4b-04f726d099c9"
+      (reference "U13") (unit 1) (value "PinVis") (footprint "")
+    )
+    (path "/c1696530-30e9-4af4-9fcd-59e8cab28548"
+      (reference "U14") (unit 1) (value "PinVis") (footprint "")
+    )
+    (path "/3c7def11-0301-4ee0-9763-7a800a47ccb5"
+      (reference "U15") (unit 1) (value "PinVis") (footprint "")
+    )
+    (path "/b364135e-c5d3-4ae8-be89-ca9a24a910d3"
+      (reference "U16") (unit 1) (value "LotsOfPins") (footprint "")
+    )
     (path "/337b2738-ac74-46e4-af99-edf86290f598"
-      (reference "U?") (unit 1) (value "LotsOfPins") (footprint "")
+      (reference "U17") (unit 1) (value "LotsOfPins") (footprint "")
+    )
+    (path "/19a2d2d0-82c9-4be0-9af0-4fc0c28dda76"
+      (reference "U18") (unit 1) (value "PinVis") (footprint "")
     )
     (path "/a5b0d54e-9873-4c04-8e3b-2303e065a341"
-      (reference "U?") (unit 1) (value "LotsOfPins") (footprint "")
-    )
-    (path "/b364135e-c5d3-4ae8-be89-ca9a24a910d3"
-      (reference "U?") (unit 1) (value "LotsOfPins") (footprint "")
-    )
-  )
+      (reference "U19") (unit 1) (value "LotsOfPins") (footprint "")
+    )
+  )
